Commit message: Update shoulder lower limit to safe value when mounted on AMR

File: interbotix_ros_manipulators/interbotix_ros_xsarms/interbotix_xsarm_descriptions/urdf/px100.urdf.xacro (robot description, xacro)
@@ -25,5 +25,5 @@
   <xacro:property name="waist_limit_vel"            value="${pi}"/>
   <xacro:property name="shoulder_limit_effort"      value="2"/>
-  <xacro:property name="shoulder_limit_lower"       value="${radians(-111)}"/>
+  <xacro:property name="shoulder_limit_lower"       value="${radians(-88)}"/>
   <xacro:property name="shoulder_limit_upper"       value="${radians(107)}"/>
   <xacro:property name="shoulder_limit_vel"         value="${pi}"/>
