Commit message: Update px100.srdf.xacro to mounted sleeping pose

File: interbotix_ros_manipulators/interbotix_ros_xsarms/interbotix_xsarm_moveit/config/srdf/px100.srdf.xacro (robot description, xacro)
@@ -43,8 +43,8 @@
     </group_state>
     <group_state name="Sleep" group="interbotix_arm">
-        <joint name="elbow" value="1.5" />
-        <joint name="shoulder" value="-1.88" />
+        <joint name="elbow" value="1.6" />
+        <joint name="shoulder" value="-1.53" />
         <joint name="waist" value="0" />
-        <joint name="wrist_angle" value="0.8" />
+        <joint name="wrist_angle" value="0.61" />
     </group_state>
     <group_state name="Released" group="interbotix_gripper">
